File: stm32 f103.kicad_sch (KiCad schematic)
At the start: 36 parts, among them J1 USB_C_Receptacle_USB2.0_14P, SW1 SW_Push, SW2 SW_SPDT, U1 STM32F103C6Tx, U2 PAC1934x-xJ6CX, U4 USBLC6-2SC6, U5 LD3985M33R_SOT23, U6 MCP2551-I-P, Y1 16Mhz

Commit message: schematic done
Parts:
- added C17, C18: 560pF, Package_TO_SOT_SMD:SOT-23-5, symbol Device:C_Small
- added C19: 0.1uF, Package_TO_SOT_SMD:SOT-23-5, symbol Device:C_Small
- added D2, D3, D4: LED, Package_DIP:DIP-8_W7.62mm, symbol Device:LED
- added J2: Screw_Terminal_01x02, Connector:Tag-Connect_TC2050-IDC-NL_2x05_P1.27mm_Vertical, symbol Connector:Screw_Terminal_01x02
- added J3: Screw_Terminal_01x12, symbol Connector:Screw_Terminal_01x12
- added J4: Screw_Terminal_01x14, symbol Connector:Screw_Terminal_01x14
- added R11: 4k7, symbol Device:R_Small
- added R12, R13: 100R, symbol Device:R_Small
- added R14: 120R, symbol Device:R_Small
- added R15, R16, R17, R18, R19, R20, R21, R22: 0R, symbol Device:R_Small
- added R23, R24, R25, R26: 0.004R, Package_DIP:DIP-8_W7.62mm, symbol Device:R_Small
- added R27: 499R, Package_DIP:DIP-8_W7.62mm, symbol Device:R_Small
- added R28: 82R, Package_DIP:DIP-8_W7.62mm, symbol Device:R_Small
- added R29: 33R, Package_DIP:DIP-8_W7.62mm, symbol Device:R_Small
- added R7: 150R, Package_DIP:DIP-8_W7.62mm, symbol Device:R_Small
Connections:
- net +3.3V: now also U2.A4 (V_{DD}), U2.B2 (V_{DD}IO), U6.3 (VDD), C19.1
- net +5V: now also J2.2 (Pin_2), R7.1; no longer U6.3 (VDD)
- net CAN_RX: now also U6.4 (RXD)
- net CAN_TX: now also U6.1 (TXD)
- net GND: now also U2.B4 (GND), U6.2 (VSS), C17.2, C18.2, C19.2, D2.1 (K), D3.1 (K), D4.1 (K), J2.1 (Pin_1), R11.2, R27.2
- net IN1+: now also R15.1, R23.1; no longer U2.A3 (SENSE1+)
- net IN1-: now also R16.1, R23.2; no longer U2.A2 (SENSE1-)
- net IN2+: now also R17.1, R24.1; no longer U2.A1 (SENSE2+)
- net IN2-: now also R18.1, R24.2; no longer U2.B1 (SENSE2-)
- net IN3+: now also R19.1, R25.1; no longer U2.D1 (SENSE3+)
- net IN4+: now also R21.1, R26.1; no longer U2.D3 (SENSE4+)
- net IN4-: now also R22.1, R26.2; no longer U2.D2 (SENSE4-)
- net SPI2_MISO: now also U1.16 (PA6), J4.8 (Pin_8); no longer U1.27 (PB14)
- net SPI2_MOSI: now also U1.17 (PA7), J4.7 (Pin_7); no longer U1.28 (PB15)
- net SPI2_SCK: now also U1.15 (PA5)
- net SPI2_SCK_B: now also J4.9 (Pin_9); no longer U1.26 (PB13)
- net PA0: now reaches U1.10 (PA0)
- net PA0: now also J4.14 (Pin_14)
- net PA1: now reaches U1.11 (PA1)
- net PA1: now also J4.13 (Pin_13)
- net PA2: now reaches U1.12 (PA2)
- net PA2: now also J4.12 (Pin_12)
- net PA3: now reaches U1.13 (PA3)
- net PA3: now also J4.11 (Pin_11)
- net PA4: now reaches U1.14 (PA4)
- net PA4: now also J4.10 (Pin_10)
- net PB0: now reaches U1.18 (PB0)
- net PB0: now also U2.C3 (SLOW)
- net PB1: now reaches U1.19 (PB1)
- net PB1: now also J3.11 (Pin_11), J3.12 (Pin_12)
- net LED_R: now reaches U1.2 (PC13)
- net LED_R: now also R28.1
- net PB2: now reaches U1.20 (PB2)
- net PB2: now also J3.10 (Pin_10)
- net PB10: now reaches U1.21 (PB10)
- net PB10: now also J3.6 (Pin_6)
- net PB11: now reaches U1.22 (PB11)
- net PB11: now also J3.5 (Pin_5)
- net PB12: now reaches U1.25 (PB12)
- net PB12: now also J3.4 (Pin_4)
- net PA8: now reaches U1.29 (PA8)
- net PA8: now also J4.6 (Pin_6)
- net LED_G: now reaches U1.3 (PC14)
- net LED_G: now also R29.1
- net USART1_TX: now reaches U1.30 (PA9)
- net USART1_TX: now also J4.5 (Pin_5)
- net USART1_RX: now reaches U1.31 (PA10)
- net USART1_RX: now also J4.4 (Pin_4)
- net PA13: now reaches U1.34 (PA13)
- net PA13: now also J4.3 (Pin_3)
- net PA14: now reaches U1.37 (PA14)
- net PA14: now also J4.2 (Pin_2)
- net PA15: now reaches U1.38 (PA15)
- net PA15: now also J4.1 (Pin_1)
- net PB3: now reaches U1.39 (PB3)
- net PB3: now also J3.9 (Pin_9)
- net PC15: now reaches U1.4 (PC15)
- net PC15: now also U2.B3 (~{PWRDN})
- net PB4: now reaches U1.40 (PB4)
- net PB4: now also J3.8 (Pin_8)
- net PB5: now reaches U1.41 (PB5)
- net PB5: now also J3.7 (Pin_7)
- net CANL: now reaches U6.6 (CANL)
- net CANL: now also R12.1, R14.2
- net CAN JUMP2: now reaches U6.7 (CANH)
- net CAN JUMP2: now also R13.1
- net at U6.8 (Rs): now also R11.1
- net at U2.C2 (ADDRSEL): now also R27.1
- net IN3_: no longer names the net of U2.C1 (SENSE3-)
- net IN3_: now also R20.2
- new net: C17.1, R12.2
- new net: D4.2 (A), R29.2
- new net: D2.2 (A), R7.2
- new net: R15.2, U2.A3 (SENSE1+)
- new net: R18.2, U2.B1 (SENSE2-)
- new net: C18.1, R13.2
- new net: R22.2, U2.D2 (SENSE4-)
- new net: D3.2 (A), R28.2
- new net: R17.2, U2.A1 (SENSE2+)
- new net: R19.2, U2.D1 (SENSE3+)
- new net: R16.2, U2.A2 (SENSE1-)
- new net: R21.2, U2.D3 (SENSE4+)
- new net CAN JUMP1: R14.1
- new net IN3-: R20.1, R25.2
- new net PB13: J3.3 (Pin_3), U1.26 (PB13)
- new net PB14: J3.2 (Pin_2), U1.27 (PB14)
- new net PB15: J3.1 (Pin_1), U1.28 (PB15)
Other:
- note added: "CAN TRANSIVER"
- note added: "CONNECTOR"
- note added: "PAC1934 VOLTAGE SENSE"
- moved on the sheet: C12, C13, C14, C15, C16, D1, J1, R10, R5, R6, R8, R9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

Commit message: git ignore for kicad
Parts:
- C1, C10, C11, C2, C3, C4, C5, C6, C7, C8, C9: footprint Package_SO:SOIC-8_3.9x4.9mm_P1.27mm -> Capacitor_SMD:C_1206_3216Metric
- C12, C13, C14, C15, C16, C17, C18, C19: footprint Package_TO_SOT_SMD:SOT-23-5 -> Capacitor_SMD:C_1206_3216Metric
- D1: footprint Diode_THT:D_DO-41_SOD81_P10.16mm_Horizontal -> Diode_SMD:D_1206_3216Metric
- D2, D3, D4: footprint Package_DIP:DIP-8_W7.62mm -> LED_SMD:LED_1210_3225Metric
- FB1, R1, R11, R12, R13, R14, R15, R16, R17, R18, R19, R2, R20, R21, R22, R3, R4: footprint (none) -> Resistor_SMD:R_1206_3216Metric
- J1: footprint (none) -> Connector_USB:USB_C_Receptacle_GCT_USB4115-03-C
- J2: footprint Connector:Tag-Connect_TC2050-IDC-NL_2x05_P1.27mm_Vertical -> Connector_Phoenix_MC:PhoenixContact_MCV_1,5_2-G-3.5_1x02_P3.50mm_Vertical
- J3: footprint (none) -> Connector_Phoenix_MC:PhoenixContact_MCV_1,5_12-G-3.5_1x12_P3.50mm_Vertical
- J4: footprint (none) -> Connector_Phoenix_MC:PhoenixContact_MCV_1,5_14-G-3.5_1x14_P3.50mm_Vertical
- R10, R23, R24, R25, R26, R27, R28, R29, R5, R6, R7, R8, R9: footprint Package_DIP:DIP-8_W7.62mm -> Resistor_SMD:R_1206_3216Metric
- SW1: footprint Button_Switch_SMD:Nidec_Copal_CAS-120A -> Button_Switch_SMD:SW_Push_1P1T_NO_Vertical_Wuerth_434133025816
- SW2: footprint Button_Switch_SMD:Nidec_Copal_CAS-120A -> Button_Switch_SMD:SW_SPDT_PCM12
- Y1: footprint (none) -> Crystal:Crystal_SMD_3225-4Pin_3.2x2.5mm
Changed lines of the file:
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@@
 			)
 		)
-		(property "Footprint" "Package_DIP:DIP-8_W7.62mm"
+		(property "Footprint" "Resistor_SMD:R_1206_3216Metric"
 			(at 50.8 196.85 0)
 			(hide yes)
@@
 			)
 		)
-		(property "Footprint" "Button_Switch_SMD:Nidec_Copal_CAS-120A"
+		(property "Footprint" "Button_Switch_SMD:SW_SPDT_PCM12"
 			(at 91.44 59.69 0)
 			(hide yes)
@@
 			)
 		)
-		(property "Footprint" "Package_DIP:DIP-8_W7.62mm"
+		(property "Footprint" "Resistor_SMD:R_1206_3216Metric"
 			(at 189.23 226.06 0)
 			(hide yes)
@@
 			)
 		)
-		(property "Footprint" ""
+		(property "Footprint" "Resistor_SMD:R_1206_3216Metric"
 			(at 240.03 68.58 0)
 			(hide yes)
@@
 			)
 		)
-		(property "Footprint" ""
+		(property "Footprint" "Resistor_SMD:R_1206_3216Metric"
 			(at 82.55 92.71 0)
 			(hide yes)
@@
 			)
 		)
-		(property "Footprint" "Package_TO_SOT_SMD:SOT-23-5"
+		(property "Footprint" "Capacitor_SMD:C_1206_3216Metric"
 			(at 273.05 71.12 0)
 			(hide yes)
@@
 			)
 		)
-		(property "Footprint" "Package_SO:SOIC-8_3.9x4.9mm_P1.27mm"
+		(property "Footprint" "Capacitor_SMD:C_1206_3216Metric"
 			(at 152.4 39.37 0)
 			(hide yes)
@@
 			)
 		)
-		(property "Footprint" ""
+		(property "Footprint" "Resistor_SMD:R_1206_3216Metric"
 			(at 273.05 64.77 0)
 			(hide yes)
@@
 			)
 		)
-		(property "Footprint" "Package_DIP:DIP-8_W7.62mm"
+		(property "Footprint" "Resistor_SMD:R_1206_3216Metric"
 			(at 50.8 220.98 0)
 			(hide yes)
@@
 			)
 		)
-		(property "Footprint" "Package_DIP:DIP-8_W7.62mm"
+		(property "Footprint" "LED_SMD:LED_1210_3225Metric"
 			(at 194.31 125.73 0)
 			(hide yes)
@@
 			)
 		)
-		(property "Footprint" "Package_DIP:DIP-8_W7.62mm"
+		(property "Footprint" "Resistor_SMD:R_1206_3216Metric"
 			(at 313.69 50.8 0)
 			(hide yes)
@@
 			)
 		)
-		(property "Footprint" "Package_DIP:DIP-8_W7.62mm"
+		(property "Footprint" "Resistor_SMD:R_1206_3216Metric"
 			(at 189.23 228.6 0)
 			(hide yes)
@@
 			)
 		)
-		(property "Footprint" "Package_SO:SOIC-8_3.9x4.9mm_P1.27mm"
+		(property "Footprint" "Capacitor_SMD:C_1206_3216Metric"
 			(at 71.12 39.37 0)
 			(hide yes)
@@
 			)
 		)
-		(property "Footprint" "Package_TO_SOT_SMD:SOT-23-5"
+		(property "Footprint" "Capacitor_SMD:C_1206_3216Metric"
 			(at 378.46 59.69 0)
 			(hide yes)
@@
 			)
 		)
-		(property "Footprint" ""
+		(property "Footprint" "Resistor_SMD:R_1206_3216Metric"
 			(at 77.47 219.71 0)
 			(hide yes)
@@
 			)
 		)
-		(property "Footprint" "Connector:Tag-Connect_TC2050-IDC-NL_2x05_P1.27mm_Vertical"
+		(property "Footprint" "Connector_Phoenix_MC:PhoenixContact_MCV_1,5_2-G-3.5_1x02_P3.50mm_Vertical"
 			(at 278.13 121.92 0)
 			(hide yes)
@@
 			)
 		)
-		(property "Footprint" ""
+		(property "Footprint" "Resistor_SMD:R_1206_3216Metric"
 			(at 77.47 201.93 0)
 			(hide yes)
@@
 			)
 		)
-		(property "Footprint" ""
+		(property "Footprint" "Connector_Phoenix_MC:PhoenixContact_MCV_1,5_14-G-3.5_1x14_P3.50mm_Vertical"
 			(at 321.31 147.32 0)
 			(hide yes)
@@
 			)
 		)
-		(property "Footprint" ""
+		(property "Footprint" "Resistor_SMD:R_1206_3216Metric"
 			(at 158.75 67.31 0)
 			(hide yes)
@@
 			)
 		)
-		(property "Footprint" "Package_SO:SOIC-8_3.9x4.9mm_P1.27mm"
+		(property "Footprint" "Capacitor_SMD:C_1206_3216Metric"
 			(at 62.23 91.44 0)
 			(hide yes)
@@
 			)
 		)
-		(property "Footprint" "Package_SO:SOIC-8_3.9x4.9mm_P1.27mm"
+		(property "Footprint" "Capacitor_SMD:C_1206_3216Metric"
 			(at 176.53 39.37 0)
 			(hide yes)
@@
 			)
 		)
-		(property "Footprint" "Package_SO:SOIC-8_3.9x4.9mm_P1.27mm"
+		(property "Footprint" "Capacitor_SMD:C_1206_3216Metric"
 			(at 41.91 91.44 0)
 			(hide yes)
@@
 			)
 		)
-		(property "Footprint" "Package_DIP:DIP-8_W7.62mm"
+		(property "Footprint" "Resistor_SMD:R_1206_3216Metric"
 			(at 50.8 234.95 0)
 			(hide yes)
@@
 			)
 		)
-		(property "Footprint" ""
+		(property "Footprint" "Resistor_SMD:R_1206_3216Metric"
 			(at 77.3839 212.09 0)
 			(hide yes)
@@
 			)
 		)
-		(property "Footprint" "Package_DIP:DIP-8_W7.62mm"
+		(property "Footprint" "Resistor_SMD:R_1206_3216Metric"
 			(at 190.5 213.36 0)
 			(hide yes)
@@
 			)
 		)
-		(property "Footprint" "Package_DIP:DIP-8_W7.62mm"
+		(property "Footprint" "Resistor_SMD:R_1206_3216Metric"
 			(at 50.8 208.28 0)
 			(hide yes)
@@
 			)
 		)
-		(property "Footprint" ""
+		(property "Footprint" "Resistor_SMD:R_1206_3216Metric"
 			(at 100.33 59.69 0)
 			(hide yes)
@@
 			)
 		)
-		(property "Footprint" "Package_DIP:DIP-8_W7.62mm"
+		(property "Footprint" "Resistor_SMD:R_1206_3216Metric"
 			(at 190.5 218.44 0)
 			(hide yes)
@@
 			)
 		)
-		(property "Footprint" "Package_TO_SOT_SMD:SOT-23-5"
+		(property "Footprint" "Capacitor_SMD:C_1206_3216Metric"
 			(at 364.49 59.69 0)
 			(hide yes)
@@
 			)
 		)
-		(property "Footprint" ""
+		(property "Footprint" "Resistor_SMD:R_1206_3216Metric"
 			(at 276.86 45.72 0)
 			(hide yes)
@@
 			)
 		)
-		(property "Footprint" ""
+		(property "Footprint" "Connector_USB:USB_C_Receptacle_GCT_USB4115-03-C"
 			(at 209.55 218.44 0)
 			(hide yes)
@@
 			)
 		)
-		(property "Footprint" "Package_SO:SOIC-8_3.9x4.9mm_P1.27mm"
+		(property "Footprint" "Capacitor_SMD:C_1206_3216Metric"
 			(at 140.97 39.37 0)
 			(hide yes)
@@
 			)
 		)
-		(property "Footprint" "Package_SO:SOIC-8_3.9x4.9mm_P1.27mm"
+		(property "Footprint" "Capacitor_SMD:C_1206_3216Metric"
 			(at 91.44 39.37 0)
 			(hide yes)
@@
 			)
 		)
-		(property "Footprint" "Package_SO:SOIC-8_3.9x4.9mm_P1.27mm"
+		(property "Footprint" "Capacitor_SMD:C_1206_3216Metric"
 			(at 73.66 59.69 0)
 			(hide yes)
@@
 			)
 		)
-		(property "Footprint" "Package_TO_SOT_SMD:SOT-23-5"
+		(property "Footprint" "Capacitor_SMD:C_1206_3216Metric"
 			(at 281.94 71.12 0)
 			(hide yes)
@@
 			)
 		)
-		(property "Footprint" ""
+		(property "Footprint" "Resistor_SMD:R_1206_3216Metric"
 			(at 77.47 227.33 0)
 			(hide yes)
@@
 			)
 		)
-		(property "Footprint" "Package_SO:SOIC-8_3.9x4.9mm_P1.27mm"
+		(property "Footprint" "Capacitor_SMD:C_1206_3216Metric"
 			(at 81.28 39.37 0)
 			(hide yes)
@@
 			)
 		)
-		(property "Footprint" "Package_DIP:DIP-8_W7.62mm"
+		(property "Footprint" "LED_SMD:LED_1210_3225Metric"
 			(at 180.34 125.73 0)
 			(hide yes)
@@
 			)
 		)
-		(property "Footprint" ""
+		(property "Footprint" "Resistor_SMD:R_1206_3216Metric"
 			(at 77.47 209.55 0)
 			(hide yes)
@@
 			)
 		)
-		(property "Footprint" ""
+		(property "Footprint" "Resistor_SMD:R_1206_3216Metric"
 			(at 73.66 92.71 0)
 			(hide yes)
@@
 			)
 		)
-		(property "Footprint" ""
+		(property "Footprint" "Connector_Phoenix_MC:PhoenixContact_MCV_1,5_12-G-3.5_1x12_P3.50mm_Vertical"
 			(at 278.13 149.86 0)
 			(hide yes)
@@
 			)
 		)
-		(property "Footprint" "Button_Switch_SMD:Nidec_Copal_CAS-120A"
+		(property "Footprint" "Button_Switch_SMD:SW_Push_1P1T_NO_Vertical_Wuerth_434133025816"
 			(at 55.88 59.69 0)
 			(hide yes)
@@
 			)
 		)
-		(property "Footprint" "Package_SO:SOIC-8_3.9x4.9mm_P1.27mm"
+		(property "Footprint" "Capacitor_SMD:C_1206_3216Metric"
 			(at 60.96 39.37 0)
 			(hide yes)
@@
 			)
 		)
-		(property "Footprint" ""
+		(property "Footprint" "Resistor_SMD:R_1206_3216Metric"
 			(at 77.47 217.17 0)
 			(hide yes)
@@
 			)
 		)
-		(property "Footprint" ""
+		(property "Footprint" "Resistor_SMD:R_1206_3216Metric"
 			(at 165.1 38.608 90)
 			(hide yes)
@@
 			)
 		)
-		(property "Footprint" "Package_DIP:DIP-8_W7.62mm"
+		(property "Footprint" "Resistor_SMD:R_1206_3216Metric"
 			(at 184.15 204.47 0)
 			(hide yes)
@@
 			)
 		)
-		(property "Footprint" "Package_SO:SOIC-8_3.9x4.9mm_P1.27mm"
+		(property "Footprint" "Capacitor_SMD:C_1206_3216Metric"
 			(at 101.6 39.37 0)
 			(hide yes)
@@
 			)
 		)
-		(property "Footprint" ""
+		(property "Footprint" "Crystal:Crystal_SMD_3225-4Pin_3.2x2.5mm"
 			(at 53.34 82.55 0)
 			(hide yes)
@@
 			)
 		)
-		(property "Footprint" ""
+		(property "Footprint" "Resistor_SMD:R_1206_3216Metric"
 			(at 77.47 204.47 0)
 			(hide yes)
@@
 			)
 		)
-		(property "Footprint" "Package_DIP:DIP-8_W7.62mm"
+		(property "Footprint" "LED_SMD:LED_1210_3225Metric"
 			(at 313.69 58.42 0)
 			(hide yes)
@@
 			)
 		)
-		(property "Footprint" "Package_TO_SOT_SMD:SOT-23-5"
+		(property "Footprint" "Capacitor_SMD:C_1206_3216Metric"
 			(at 393.7 59.69 0)
 			(hide yes)
@@
 			)
 		)
-		(property "Footprint" "Package_TO_SOT_SMD:SOT-23-5"
+		(property "Footprint" "Capacitor_SMD:C_1206_3216Metric"
 			(at 337.82 59.69 0)
 			(hide yes)
@@
 			)
 		)
-		(property "Footprint" "Package_TO_SOT_SMD:SOT-23-5"
+		(property "Footprint" "Capacitor_SMD:C_1206_3216Metric"
 			(at 325.12 54.61 0)
 			(hide yes)
@@
 			)
 		)
-		(property "Footprint" "Package_TO_SOT_SMD:SOT-23-5"
+		(property "Footprint" "Capacitor_SMD:C_1206_3216Metric"
 			(at 270.51 35.56 0)
 			(hide yes)
@@
 			)
 		)
-		(property "Footprint" "Diode_THT:D_DO-41_SOD81_P10.16mm_Horizontal"
+		(property "Footprint" "Diode_SMD:D_1206_3216Metric"
 			(at 181.61 238.125 0)
 			(hide yes)
@@
 			)
 		)
-		(property "Footprint" "Package_DIP:DIP-8_W7.62mm"
+		(property "Footprint" "Resistor_SMD:R_1206_3216Metric"
 			(at 180.34 119.38 0)
 			(hide yes)
@@
 			)
 		)
-		(property "Footprint" "Package_DIP:DIP-8_W7.62mm"
+		(property "Footprint" "Resistor_SMD:R_1206_3216Metric"
 			(at 118.11 224.79 0)
 			(hide yes)
@@
 			)
 		)
-		(property "Footprint" ""
+		(property "Footprint" "Resistor_SMD:R_1206_3216Metric"
 			(at 281.94 64.77 0)
 			(hide yes)
@@
 			)
 		)
-		(property "Footprint" "Package_DIP:DIP-8_W7.62mm"
+		(property "Footprint" "Resistor_SMD:R_1206_3216Metric"
 			(at 194.31 119.38 0)
 			(hide yes)
@@
 			)
 		)
-		(property "Footprint" ""
+		(property "Footprint" "Resistor_SMD:R_1206_3216Metric"
 			(at 77.47 224.79 0)
 			(hide yes)

Commit message: v0.1
Parts:
- added J5: Screw_Terminal_01x04, symbol Connector:Screw_Terminal_01x04
- added J6: Screw_Terminal_01x08, symbol Connector:Screw_Terminal_01x08
Connections:
- net CAN JUMP1: now also J5.3 (Pin_3)
- net CAN JUMP2: now also J5.2 (Pin_2), J5.4 (Pin_4)
- net CANL: now also J5.1 (Pin_1)
- net IN1+: now also J6.8 (Pin_8)
- net IN1-: now also J6.7 (Pin_7)
- net IN2+: now also J6.6 (Pin_6)
- net IN2-: now also J6.5 (Pin_5)
- net IN3+: now also J6.4 (Pin_4)
- net IN3-: now also J6.3 (Pin_3)
- net IN4+: now also J6.2 (Pin_2)
- net IN4-: now also J6.1 (Pin_1)
- no-connect marks 0 -> 1
Other:
- moved on the sheet: J2, J3, J4

Commit message: final sch
Parts:
- J5: footprint (none) -> Connector_Phoenix_MC:PhoenixContact_MCV_1,5_4-G-3.5_1x04_P3.50mm_Vertical
- J6: footprint (none) -> Connector_Phoenix_MC:PhoenixContact_MCV_1,5_8-G-3.81_1x08_P3.81mm_Vertical
Changed lines of the file:
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@@
 			)
 		)
-		(property "Footprint" ""
+		(property "Footprint" "Connector_Phoenix_MC:PhoenixContact_MCV_1,5_8-G-3.81_1x08_P3.81mm_Vertical"
 			(at 284.48 199.39 0)
 			(hide yes)
@@
 			)
 		)
-		(property "Footprint" ""
+		(property "Footprint" "Connector_Phoenix_MC:PhoenixContact_MCV_1,5_4-G-3.5_1x04_P3.50mm_Vertical"
 			(at 341.63 198.12 0)
 			(hide yes)

Commit message: for ic going for new file
Other:
- moved on the sheet: R15, R16, R17, R18, R19, R20, R21, R22, R23, R24, R25, R26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
